Commit message: modify urdf.xacro for gazebo simulation

File: aero_description/typeF/robots/aero.urdf.xacro (robot description, xacro)
@@ -15,3 +15,9 @@
  <xacro:aero-upper/>
  <xacro:aero-wheels base_link="base_link"/>
+  <gazebo>
+   <plugin name="gazebo_ros_control" filename="libgazebo_ros_control.so">
+     <robotNamespace>/AeroUpperRobot</robotNamespace>
+     <robotSimType>gazebo_ros_control/DefaultRobotHWSim</robotSimType>
+   </plugin>
+ </gazebo>
 </robot>

File: aero_shop/trx_s/urdf/trx_s.urdf.xacro (robot description, xacro)
@@ -48,7 +48,7 @@
     </collision> </xacro:unless>
     <inertial>
-      <mass value="0" />
-      <origin xyz="0 0 0" rpy="0 -0 0"/>
-      <inertia ixx="0" ixy="0" ixz="0" iyy="0" iyz="0" izz="0"/>
+      <mass value="0.001" />
+      <origin xyz="0 0 0" rpy="0 -0 0"/>
+      <inertia ixx="0.001" ixy="0" ixz="0" iyy="0.001" iyz="0" izz="0.001"/>
     </inertial>
   </link>
@@ -71,7 +71,7 @@
     </collision> </xacro:unless>
     <inertial>
-      <mass value="0" />
-      <origin xyz="0 0 0" rpy="0 -0 0"/>
-      <inertia ixx="0" ixy="0" ixz="0" iyy="0" iyz="0" izz="0"/>
+      <mass value="0.001" />
+      <origin xyz="0 0 0" rpy="0 -0 0"/>
+      <inertia ixx="0.001" ixy="0" ixz="0" iyy="0.001" iyz="0" izz="0.001"/>
     </inertial>
   </link>
@@ -94,7 +94,7 @@
     </collision> </xacro:unless>
     <inertial>
-      <mass value="0" />
-      <origin xyz="0 0 0" rpy="0 -0 0"/>
-      <inertia ixx="0" ixy="0" ixz="0" iyy="0" iyz="0" izz="0"/>
+      <mass value="0.001" />
+      <origin xyz="0 0 0" rpy="0 -0 0"/>
+      <inertia ixx="0.001" ixy="0" ixz="0" iyy="0.001" iyz="0" izz="0.001"/>
     </inertial>
   </link>
@@ -117,7 +117,7 @@
     </collision> </xacro:unless>
     <inertial>
-      <mass value="0" />
-      <origin xyz="0 0 0" rpy="0 -0 0"/>
-      <inertia ixx="0" ixy="0" ixz="0" iyy="0" iyz="0" izz="0"/>
+      <mass value="0.001" />
+      <origin xyz="0 0 0" rpy="0 -0 0"/>
+      <inertia ixx="0.001" ixy="0" ixz="0" iyy="0.001" iyz="0" izz="0.001"/>
     </inertial>
   </link>
@@ -156,8 +156,13 @@
     <dynamics damping="0.2" friction="0" />
   </joint>
-  <transmission type="pr2_mechanism_model/SimpleTransmission" name="${prefix}_indexend_joint_trans" >
-    <actuator name="${prefix}_indexend_joint_motor" />
-    <joint name="${prefix}_indexend_joint" />
-    <mechanicalReduction>1</mechanicalReduction>
+  <transmission name="${prefix}_indexend_joint_trans">
+    <type>transmission_interface/SimpleTransmission</type>
+    <joint name="${prefix}_indexend_joint">
+      <hardwareInterface>hardware_interface/EffortJointInterface</hardwareInterface>
+    </joint>
+    <actuator name="${prefix}_indexend_joint_motor">
+      <hardwareInterface>hardware_interface/EffortJointInterface</hardwareInterface>
+      <mechanicalReduction>1</mechanicalReduction>
+    </actuator>
   </transmission>
   <gazebo reference="${prefix}_indexend_joint">
@@ -172,8 +177,13 @@
     <dynamics damping="0.2" friction="0" />
   </joint>
-  <transmission type="pr2_mechanism_model/SimpleTransmission" name="${prefix}_thumb_joint_trans" >
-    <actuator name="${prefix}_thumb_joint_motor" />
-    <joint name="${prefix}_thumb_joint" />
-    <mechanicalReduction>1</mechanicalReduction>
+  <transmission name="${prefix}_thumb_joint_trans">
+    <type>transmission_interface/SimpleTransmission</type>
+    <joint name="${prefix}_thumb_joint">
+      <hardwareInterface>hardware_interface/EffortJointInterface</hardwareInterface>
+    </joint>
+    <actuator name="${prefix}_thumb_joint_motor">
+      <hardwareInterface>hardware_interface/EffortJointInterface</hardwareInterface>
+      <mechanicalReduction>1</mechanicalReduction>
+    </actuator>
   </transmission>
   <gazebo reference="${prefix}_thumb_joint">

File: aero_shop/typeC_lifter/urdf/lifter.urdf.xacro (robot description, xacro)
@@ -41,11 +41,11 @@
     <link name="leg_foreleg_link">
       <visual>
-        <origin xyz="0.0 0.0 0" rpy="3.1415 -0 0"/>
-        <geometry>
-          <mesh filename="package://aero_description/meshes/typeC_lifter/lifter_bone.dae" scale="1 1 1" />
-        </geometry>
-      </visual>
-      <collision>
-        <origin xyz="0.0 0.0 0.0" rpy="0 -0 0"/>
+        <origin xyz="0.0 0.0 0.0" rpy="3.1415 -0 0"/>
+        <geometry>
+          <mesh filename="package://aero_description/meshes/typeC_lifter/lifter_bone.dae" scale="1 1 1" />
+       </geometry>
+      </visual>
+      <collision>
+        <origin xyz="0.0 0.0 0.0" rpy="3.1415 -0 0"/>
         <geometry>
           <mesh filename="package://aero_description/meshes/typeC_lifter/lifter_bone.dae" scale="1 1 1" />
@@ -64,5 +64,5 @@
     <link name="leg_knee_link">
       <visual>
-        <origin xyz="0.0 0.0 0" rpy="3.1415 -0 0"/>
+        <origin xyz="0.0 0.0 0.0" rpy="3.1415 -0 0"/>
         <geometry>
           <mesh filename="package://aero_description/meshes/typeC_lifter/lifter_knee.dae" scale="1 1 1" />
@@ -70,5 +70,5 @@
       </visual>
       <collision>
-        <origin xyz="0.0 0.0 0.0" rpy="0 -0 0"/>
+        <origin xyz="0.0 0.0 0.0" rpy="3.1415 -0 0"/>
         <geometry>
           <mesh filename="package://aero_description/meshes/typeC_lifter/lifter_knee.dae" scale="1 1 1" />
@@ -93,5 +93,5 @@
       </visual>
       <collision>
-        <origin xyz="0.0 0.0 0.0" rpy="0 -0 0"/>
+        <origin xyz="0.0 0.0 0.25" rpy="0 -0 0"/>
         <geometry>
           <mesh filename="package://aero_description/meshes/typeC_lifter/lifter_bone.dae" scale="1 1 1" />
@@ -116,5 +116,5 @@
       </visual>
       <collision>
-        <origin xyz="0 0 0" rpy="0 -0 0"/>
+        <origin xyz="0 0 0.05" rpy="3.1415920 0 0"/>
         <geometry>
           <mesh filename="package://aero_description/meshes/typeC_lifter/lifter_base.dae" scale="1 1 1" />
@@ -164,12 +164,17 @@
       <origin xyz="0 0 0.25" rpy="0 0 0"/>
       <axis   xyz="0 -1 0"/>
-      <limit lower="0" upper="1.5707" effort="100" velocity="0.5" />
+      <limit lower="0" upper="1.5707" effort="1000" velocity="0.5" />
       <dynamics damping="0.2" friction="0" />
     </joint>
-    <transmission type="pr2_mechanism_model/SimpleTransmission" name="hip_joint_trans" >
-      <actuator name="hip_joint_motor" />
-      <joint name="hip_joint" />
+    <transmission name="hip_joint_trans">
+    <type>transmission_interface/SimpleTransmission</type>
+    <joint name="hip_joint">
+      <hardwareInterface>hardware_interface/EffortJointInterface</hardwareInterface>
+    </joint>
+    <actuator name="hip_joint_motor">
+      <hardwareInterface>hardware_interface/EffortJointInterface</hardwareInterface>
       <mechanicalReduction>1</mechanicalReduction>
-    </transmission>
+    </actuator>
+  </transmission>
     <gazebo reference="hip_joint">
       <implicitSpringDamper>0.4</implicitSpringDamper>
@@ -198,11 +203,16 @@
       <origin xyz="0 0 0.05" rpy="0 0 0"/>
       <axis   xyz="0 -1 0"/>
-      <limit lower="0" upper="1.5707" effort="100" velocity="0.5" />
+      <limit lower="0" upper="1.5707" effort="1000" velocity="0.5" />
       <dynamics damping="0.2" friction="0" />
     </joint>
-    <transmission type="pr2_mechanism_model/SimpleTransmission" name="ankle_joint_trans" >
-      <actuator name="ankle_joint_motor" />
-      <joint name="ankle_joint" />
-      <mechanicalReduction>1</mechanicalReduction>
+    <transmission name="ankle_joint_trans">
+      <type>transmission_interface/SimpleTransmission</type>
+      <joint name="ankle_joint">
+        <hardwareInterface>hardware_interface/EffortJointInterface</hardwareInterface>
+      </joint>
+      <actuator name="ankle_joint_motor">
+        <hardwareInterface>hardware_interface/EffortJointInterface</hardwareInterface>
+        <mechanicalReduction>1</mechanicalReduction>
+      </actuator>
     </transmission>
     <gazebo reference="ankle_joint">
@@ -211,17 +221,17 @@
 <!--- mimic joints -->
 <!-- requried -->
-    <joint name="knee_joint_foreleg_dummy" type="continuous">
+    <joint name="knee_joint_foreleg_dummy" type="fixed">
       <parent link="leg_foreleg_link"/>
       <child  link="leg_knee_link"/>
       <origin xyz="0 0 0.25" rpy="0 0 0"/>
       <axis   xyz="0 -1 0"/>
-      <mimic joint="ankle_joint" multiplier="-1" offset="0" />
-    </joint>
-    <joint name="knee_joint_thigh_dummy" type="continuous">
+      <!--mimic joint="ankle_joint" multiplier="-1" offset="0" /-->
+    </joint>
+    <joint name="knee_joint_thigh_dummy" type="fixed">
       <parent link="leg_knee_link"/>
       <child  link="leg_thigh_link"/>
       <origin xyz="0 0 0.12" rpy="0 0 0"/>
       <axis xyz="0 -1 0"/>
-      <mimic joint="hip_joint" multiplier="-1" offset="0" />
+      <!--mimic joint="hip_joint" multiplier="-1" offset="0" /-->
     </joint>
 <!-- redundant -->

File: aero_shop/typeD_wheel/urdf/wheels.urdf.xacro (robot description, xacro)
@@ -72,5 +72,5 @@
       </visual> </xacro:unless>
       <xacro:unless value="${disable_mesh}"> <collision>
-        <origin xyz="0.0 0.0 0.0" rpy="0 -0 0"/>
+        <origin xyz="0.0 0.0 0.0" rpy="-1.57079632679 -0 0"/>
         <geometry>
           <mesh filename="package://aero_description/meshes/typeD_wheel/wheels_mecanum.dae" scale="1 1 1" />
@@ -95,5 +95,5 @@
       </visual> </xacro:unless>
       <xacro:unless value="${disable_mesh}"> <collision>
-        <origin xyz="0.0 0.0 0.0" rpy="0 -0 0"/>
+        <origin xyz="0.0 0.0 0.0" rpy="-1.57079632679 -0 0"/>
         <geometry>
           <mesh filename="package://aero_description/meshes/typeD_wheel/wheels_mecanum.dae" scale="1 1 1" />
@@ -118,5 +118,5 @@
       </visual> </xacro:unless>
       <xacro:unless value="${disable_mesh}"> <collision>
-        <origin xyz="0.0 0.0 0.0" rpy="0 -0 0"/>
+        <origin xyz="0.0 0.0 0.0" rpy="-1.57079632679 -0 0"/>
         <geometry>
           <mesh filename="package://aero_description/meshes/typeD_wheel/wheels_mecanum.dae" scale="1 1 1" />
@@ -141,5 +141,5 @@
       </visual> </xacro:unless>
       <xacro:unless value="${disable_mesh}"> <collision>
-        <origin xyz="0.0 0.0 0.0" rpy="0 -0 0"/>
+        <origin xyz="0.0 0.0 0.0" rpy="-1.57079632679 -0 0"/>
         <geometry>
           <mesh filename="package://aero_description/meshes/typeD_wheel/wheels_mecanum.dae" scale="1 1 1" />
