Commit message: modify urdf.xacro for gazebo simulation

File: aero_shop/typeF_upperbody/urdf/aero_upper_typef.urdf.xacro (robot description, xacro)
@@ -419,8 +419,13 @@
     <dynamics damping="0.2" friction="0" />
   </joint>
-  <transmission type="pr2_mechanism_model/SimpleTransmission" name="waist_y_joint_trans" >
-    <actuator name="waist_y_joint_motor" />
-    <joint name="waist_y_joint" />
-    <mechanicalReduction>1</mechanicalReduction>
+  <transmission name="waist_y_joint_trans">
+    <type>transmission_interface/SimpleTransmission</type>
+    <joint name="waist_y_joint">
+      <hardwareInterface>hardware_interface/EffortJointInterface</hardwareInterface>
+    </joint>
+    <actuator name="waist_y_joint_motor">
+      <hardwareInterface>hardware_interface/EffortJointInterface</hardwareInterface>
+      <mechanicalReduction>1</mechanicalReduction>
+    </actuator>
   </transmission>
   <gazebo reference="waist_y_joint">
@@ -436,8 +441,13 @@
     <dynamics damping="0.2" friction="0" />
   </joint>
-  <transmission type="pr2_mechanism_model/SimpleTransmission" name="waist_p_joint_trans" >
-    <actuator name="waist_p_joint_motor" />
-    <joint name="waist_p_joint" />
-    <mechanicalReduction>1</mechanicalReduction>
+  <transmission name="waist_p_joint_trans">
+    <type>transmission_interface/SimpleTransmission</type>
+    <joint name="waist_p_joint">
+      <hardwareInterface>hardware_interface/EffortJointInterface</hardwareInterface>
+    </joint>
+    <actuator name="waist_p_joint_motor">
+      <hardwareInterface>hardware_interface/EffortJointInterface</hardwareInterface>
+      <mechanicalReduction>1</mechanicalReduction>
+    </actuator>
   </transmission>
   <gazebo reference="waist_p_joint">
@@ -453,8 +463,13 @@
     <dynamics damping="0.2" friction="0" />
   </joint>
-  <transmission type="pr2_mechanism_model/SimpleTransmission" name="waist_r_joint_trans" >
-    <actuator name="waist_r_joint_motor" />
-    <joint name="waist_r_joint" />
-    <mechanicalReduction>1</mechanicalReduction>
+  <transmission name="waist_r_joint_trans">
+    <type>transmission_interface/SimpleTransmission</type>
+    <joint name="waist_r_joint">
+      <hardwareInterface>hardware_interface/EffortJointInterface</hardwareInterface>
+    </joint>
+    <actuator name="waist_r_joint_motor">
+      <hardwareInterface>hardware_interface/EffortJointInterface</hardwareInterface>
+      <mechanicalReduction>1</mechanicalReduction>
+    </actuator>
   </transmission>
   <gazebo reference="waist_r_joint">
@@ -470,8 +485,13 @@
     <dynamics damping="0.2" friction="0" />
   </joint>
-  <transmission type="pr2_mechanism_model/SimpleTransmission" name="l_shoulder_p_joint_trans" >
-    <actuator name="l_shoulder_p_joint_motor" />
-    <joint name="l_shoulder_p_joint" />
-    <mechanicalReduction>1</mechanicalReduction>
+  <transmission name="l_shoulder_p_joint_trans">
+    <type>transmission_interface/SimpleTransmission</type>
+    <joint name="l_shoulder_p_joint">
+      <hardwareInterface>hardware_interface/EffortJointInterface</hardwareInterface>
+    </joint>
+    <actuator name="l_shoulder_p_joint_motor">
+      <hardwareInterface>hardware_interface/EffortJointInterface</hardwareInterface>
+      <mechanicalReduction>1</mechanicalReduction>
+    </actuator>
   </transmission>
   <gazebo reference="l_shoulder_p_joint">
@@ -487,8 +507,13 @@
     <dynamics damping="0.2" friction="0" />
   </joint>
-  <transmission type="pr2_mechanism_model/SimpleTransmission" name="l_shoulder_r_joint_trans" >
-    <actuator name="l_shoulder_r_joint_motor" />
-    <joint name="l_shoulder_r_joint" />
-    <mechanicalReduction>1</mechanicalReduction>
+  <transmission name="l_shoulder_r_joint_trans">
+    <type>transmission_interface/SimpleTransmission</type>
+    <joint name="l_shoulder_r_joint">
+      <hardwareInterface>hardware_interface/EffortJointInterface</hardwareInterface>
+    </joint>
+    <actuator name="l_shoulder_r_joint_motor">
+      <hardwareInterface>hardware_interface/EffortJointInterface</hardwareInterface>
+      <mechanicalReduction>1</mechanicalReduction>
+    </actuator>
   </transmission>
   <gazebo reference="l_shoulder_r_joint">
@@ -504,12 +529,18 @@
     <dynamics damping="0.2" friction="0" />
   </joint>
-  <transmission type="pr2_mechanism_model/SimpleTransmission" name="l_shoulder_y_joint_trans" >
-    <actuator name="l_shoulder_y_joint_motor" />
-    <joint name="l_shoulder_y_joint" />
-    <mechanicalReduction>1</mechanicalReduction>
+  <transmission name="l_shoulder_y_joint_trans">
+    <type>transmission_interface/SimpleTransmission</type>
+    <joint name="l_shoulder_y_joint">
+      <hardwareInterface>hardware_interface/EffortJointInterface</hardwareInterface>
+    </joint>
+    <actuator name="l_shoulder_y_joint_motor">
+      <hardwareInterface>hardware_interface/EffortJointInterface</hardwareInterface>
+      <mechanicalReduction>1</mechanicalReduction>
+    </actuator>
   </transmission>
   <gazebo reference="l_shoulder_y_joint">
     <implicitSpringDamper>0.4</implicitSpringDamper>
   </gazebo>
+  <!-- from -140 to 0 degrees-->
   <joint name="l_elbow_joint" type="revolute">
     <parent link="l_upperarm_link"/>
@@ -517,12 +548,16 @@
     <origin xyz="0.035 0 -0.1625" rpy="0 -0 0 "/>
     <axis   xyz="0 1 0"/>
-    <!-- from -140 to 0 degrees-->
     <limit lower="-2.44246" upper="0" effort="100" velocity="2.3" />
     <dynamics damping="0.2" friction="0" />
   </joint>
-  <transmission type="pr2_mechanism_model/SimpleTransmission" name="l_elbow_joint_trans" >
-    <actuator name="l_elbow_joint_motor" />
-    <joint name="l_elbow_joint" />
-    <mechanicalReduction>1</mechanicalReduction>
+  <transmission name="l_elbow_joint_trans">
+    <type>transmission_interface/SimpleTransmission</type>
+    <joint name="l_elbow_joint">
+      <hardwareInterface>hardware_interface/EffortJointInterface</hardwareInterface>
+    </joint>
+    <actuator name="l_elbow_joint_motor">
+      <hardwareInterface>hardware_interface/EffortJointInterface</hardwareInterface>
+      <mechanicalReduction>1</mechanicalReduction>
+    </actuator>
   </transmission>
   <gazebo reference="l_elbow_joint">
@@ -538,8 +573,13 @@
     <dynamics damping="0.2" friction="0" />
   </joint>
-  <transmission type="pr2_mechanism_model/SimpleTransmission" name="l_wrist_y_joint_trans" >
-    <actuator name="l_wrist_y_joint_motor" />
-    <joint name="l_wrist_y_joint" />
-    <mechanicalReduction>1</mechanicalReduction>
+  <transmission name="l_wrist_y_joint_trans">
+    <type>transmission_interface/SimpleTransmission</type>
+    <joint name="l_wrist_y_joint">
+      <hardwareInterface>hardware_interface/EffortJointInterface</hardwareInterface>
+    </joint>
+    <actuator name="l_wrist_y_joint_motor">
+      <hardwareInterface>hardware_interface/EffortJointInterface</hardwareInterface>
+      <mechanicalReduction>1</mechanicalReduction>
+    </actuator>
   </transmission>
   <gazebo reference="l_wrist_y_joint">
@@ -555,8 +595,13 @@
     <dynamics damping="0.2" friction="0" />
   </joint>
-  <transmission type="pr2_mechanism_model/SimpleTransmission" name="l_wrist_p_joint_trans" >
-    <actuator name="l_wrist_p_joint_motor" />
-    <joint name="l_wrist_p_joint" />
-    <mechanicalReduction>1</mechanicalReduction>
+  <transmission name="l_wrist_p_joint_trans">
+    <type>transmission_interface/SimpleTransmission</type>
+    <joint name="l_wrist_p_joint">
+      <hardwareInterface>hardware_interface/EffortJointInterface</hardwareInterface>
+    </joint>
+    <actuator name="l_wrist_p_joint_motor">
+      <hardwareInterface>hardware_interface/EffortJointInterface</hardwareInterface>
+      <mechanicalReduction>1</mechanicalReduction>
+    </actuator>
   </transmission>
   <gazebo reference="l_wrist_p_joint">
@@ -572,8 +617,13 @@
     <dynamics damping="0.2" friction="0" />
   </joint>
-  <transmission type="pr2_mechanism_model/SimpleTransmission" name="l_wrist_r_joint_trans" >
-    <actuator name="l_wrist_r_joint_motor" />
-    <joint name="l_wrist_r_joint" />
-    <mechanicalReduction>1</mechanicalReduction>
+  <transmission name="l_wrist_r_joint_trans">
+    <type>transmission_interface/SimpleTransmission</type>
+    <joint name="l_wrist_r_joint">
+      <hardwareInterface>hardware_interface/EffortJointInterface</hardwareInterface>
+    </joint>
+    <actuator name="l_wrist_r_joint_motor">
+      <hardwareInterface>hardware_interface/EffortJointInterface</hardwareInterface>
+      <mechanicalReduction>1</mechanicalReduction>
+    </actuator>
   </transmission>
   <gazebo reference="l_wrist_r_joint">
@@ -588,8 +638,13 @@
     <dynamics damping="0.2" friction="0" />
   </joint>
-  <transmission type="pr2_mechanism_model/SimpleTransmission" name="neck_y_joint_trans" >
-    <actuator name="neck_y_joint_motor" />
-    <joint name="neck_y_joint" />
-    <mechanicalReduction>1</mechanicalReduction>
+  <transmission name="neck_y_joint_trans">
+    <type>transmission_interface/SimpleTransmission</type>
+    <joint name="neck_y_joint">
+      <hardwareInterface>hardware_interface/EffortJointInterface</hardwareInterface>
+    </joint>
+    <actuator name="neck_y_joint_motor">
+      <hardwareInterface>hardware_interface/EffortJointInterface</hardwareInterface>
+      <mechanicalReduction>1</mechanicalReduction>
+    </actuator>
   </transmission>
   <gazebo reference="neck_y_joint">
@@ -604,8 +659,13 @@
     <dynamics damping="0.2" friction="0" />
   </joint>
-  <transmission type="pr2_mechanism_model/SimpleTransmission" name="neck_p_joint_trans" >
-    <actuator name="neck_p_joint_motor" />
-    <joint name="neck_p_joint" />
-    <mechanicalReduction>1</mechanicalReduction>
+  <transmission name="neck_p_joint_trans">
+    <type>transmission_interface/SimpleTransmission</type>
+    <joint name="neck_p_joint">
+      <hardwareInterface>hardware_interface/EffortJointInterface</hardwareInterface>
+    </joint>
+    <actuator name="neck_p_joint_motor">
+      <hardwareInterface>hardware_interface/EffortJointInterface</hardwareInterface>
+      <mechanicalReduction>1</mechanicalReduction>
+    </actuator>
   </transmission>
   <gazebo reference="neck_p_joint">
@@ -620,8 +680,13 @@
     <dynamics damping="0.2" friction="0" />
   </joint>
-  <transmission type="pr2_mechanism_model/SimpleTransmission" name="neck_r_joint_trans" >
-    <actuator name="neck_r_joint_motor" />
-    <joint name="neck_r_joint" />
-    <mechanicalReduction>1</mechanicalReduction>
+  <transmission name="neck_r_joint_trans">
+    <type>transmission_interface/SimpleTransmission</type>
+    <joint name="neck_r_joint">
+      <hardwareInterface>hardware_interface/EffortJointInterface</hardwareInterface>
+    </joint>
+    <actuator name="neck_r_joint_motor">
+      <hardwareInterface>hardware_interface/EffortJointInterface</hardwareInterface>
+      <mechanicalReduction>1</mechanicalReduction>
+    </actuator>
   </transmission>
   <gazebo reference="neck_r_joint">
@@ -637,8 +702,13 @@
     <dynamics damping="0.2" friction="0" />
   </joint>
-  <transmission type="pr2_mechanism_model/SimpleTransmission" name="r_shoulder_p_joint_trans" >
-    <actuator name="r_shoulder_p_joint_motor" />
-    <joint name="r_shoulder_p_joint" />
-    <mechanicalReduction>1</mechanicalReduction>
+  <transmission name="r_shoulder_p_joint_trans">
+    <type>transmission_interface/SimpleTransmission</type>
+    <joint name="r_shoulder_p_joint">
+      <hardwareInterface>hardware_interface/EffortJointInterface</hardwareInterface>
+    </joint>
+    <actuator name="r_shoulder_p_joint_motor">
+      <hardwareInterface>hardware_interface/EffortJointInterface</hardwareInterface>
+      <mechanicalReduction>1</mechanicalReduction>
+    </actuator>
   </transmission>
   <gazebo reference="r_shoulder_p_joint">
@@ -654,8 +724,13 @@
     <dynamics damping="0.2" friction="0" />
   </joint>
-  <transmission type="pr2_mechanism_model/SimpleTransmission" name="r_shoulder_r_joint_trans" >
-    <actuator name="r_shoulder_r_joint_motor" />
-    <joint name="r_shoulder_r_joint" />
-    <mechanicalReduction>1</mechanicalReduction>
+  <transmission name="r_shoulder_r_joint_trans">
+    <type>transmission_interface/SimpleTransmission</type>
+    <joint name="r_shoulder_r_joint">
+      <hardwareInterface>hardware_interface/EffortJointInterface</hardwareInterface>
+    </joint>
+    <actuator name="r_shoulder_r_joint_motor">
+      <hardwareInterface>hardware_interface/EffortJointInterface</hardwareInterface>
+      <mechanicalReduction>1</mechanicalReduction>
+    </actuator>
   </transmission>
   <gazebo reference="r_shoulder_r_joint">
@@ -671,8 +746,13 @@
     <dynamics damping="0.2" friction="0" />
   </joint>
-  <transmission type="pr2_mechanism_model/SimpleTransmission" name="r_shoulder_y_joint_trans" >
-    <actuator name="r_shoulder_y_joint_motor" />
-    <joint name="r_shoulder_y_joint" />
-    <mechanicalReduction>1</mechanicalReduction>
+  <transmission name="r_shoulder_y_joint_trans">
+    <type>transmission_interface/SimpleTransmission</type>
+    <joint name="r_shoulder_y_joint">
+      <hardwareInterface>hardware_interface/EffortJointInterface</hardwareInterface>
+    </joint>
+    <actuator name="r_shoulder_y_joint_motor">
+      <hardwareInterface>hardware_interface/EffortJointInterface</hardwareInterface>
+      <mechanicalReduction>1</mechanicalReduction>
+    </actuator>
   </transmission>
   <gazebo reference="r_shoulder_y_joint">
@@ -688,8 +768,13 @@
     <dynamics damping="0.2" friction="0" />
   </joint>
-  <transmission type="pr2_mechanism_model/SimpleTransmission" name="r_elbow_joint_trans" >
-    <actuator name="r_elbow_joint_motor" />
-    <joint name="r_elbow_joint" />
-    <mechanicalReduction>1</mechanicalReduction>
+  <transmission name="r_elbow_joint_trans">
+    <type>transmission_interface/SimpleTransmission</type>
+    <joint name="r_elbow_joint">
+      <hardwareInterface>hardware_interface/EffortJointInterface</hardwareInterface>
+    </joint>
+    <actuator name="r_elbow_joint_motor">
+      <hardwareInterface>hardware_interface/EffortJointInterface</hardwareInterface>
+      <mechanicalReduction>1</mechanicalReduction>
+    </actuator>
   </transmission>
   <gazebo reference="r_elbow_joint">
@@ -705,8 +790,13 @@
     <dynamics damping="0.2" friction="0" />
   </joint>
-  <transmission type="pr2_mechanism_model/SimpleTransmission" name="r_wrist_y_joint_trans" >
-    <actuator name="r_wrist_y_joint_motor" />
-    <joint name="r_wrist_y_joint" />
-    <mechanicalReduction>1</mechanicalReduction>
+  <transmission name="r_wrist_y_joint_trans">
+    <type>transmission_interface/SimpleTransmission</type>
+    <joint name="r_wrist_y_joint">
+      <hardwareInterface>hardware_interface/EffortJointInterface</hardwareInterface>
+    </joint>
+    <actuator name="r_wrist_y_joint_motor">
+      <hardwareInterface>hardware_interface/EffortJointInterface</hardwareInterface>
+      <mechanicalReduction>1</mechanicalReduction>
+    </actuator>
   </transmission>
   <gazebo reference="r_wrist_y_joint">
@@ -722,8 +812,13 @@
     <dynamics damping="0.2" friction="0" />
   </joint>
-  <transmission type="pr2_mechanism_model/SimpleTransmission" name="r_wrist_p_joint_trans" >
-    <actuator name="r_wrist_p_joint_motor" />
-    <joint name="r_wrist_p_joint" />
-    <mechanicalReduction>1</mechanicalReduction>
+  <transmission name="r_wrist_p_joint_trans">
+    <type>transmission_interface/SimpleTransmission</type>
+    <joint name="r_wrist_p_joint">
+      <hardwareInterface>hardware_interface/EffortJointInterface</hardwareInterface>
+    </joint>
+    <actuator name="r_wrist_p_joint_motor">
+      <hardwareInterface>hardware_interface/EffortJointInterface</hardwareInterface>
+      <mechanicalReduction>1</mechanicalReduction>
+    </actuator>
   </transmission>
   <gazebo reference="r_wrist_p_joint">
@@ -739,8 +834,13 @@
     <dynamics damping="0.2" friction="0" />
   </joint>
-  <transmission type="pr2_mechanism_model/SimpleTransmission" name="r_wrist_r_joint_trans" >
-    <actuator name="r_wrist_r_joint_motor" />
-    <joint name="r_wrist_r_joint" />
-    <mechanicalReduction>1</mechanicalReduction>
+  <transmission name="r_wrist_r_joint_trans">
+    <type>transmission_interface/SimpleTransmission</type>
+    <joint name="r_wrist_r_joint">
+      <hardwareInterface>hardware_interface/EffortJointInterface</hardwareInterface>
+    </joint>
+    <actuator name="r_wrist_r_joint_motor">
+      <hardwareInterface>hardware_interface/EffortJointInterface</hardwareInterface>
+      <mechanicalReduction>1</mechanicalReduction>
+    </actuator>
   </transmission>
   <gazebo reference="r_wrist_r_joint">
